File: pcb.sch (EAGLE design)
At the start: 83 parts, among them U1.1 REG101-3_DBV_5, U2.1 TCA6416A_PW_24, U4.1 TLV2242_D_8, U6.1 DCH010505S_EDJ_4, U6.2 ISO7221A_D_8, U6.3 TS5A3357_DCU_8, U6.4 TS5A3357_DCU_8, U8.1 DCH010505S_EDJ_4, U8.2 MAX232E_D_16, U8.3 ISO7221A_D_8, U9.1 DCH010505S_EDJ_4, U9.2 ISO7420Fx

Commit message: Separated Analog ground from digital ground
Connections:
- new net A_GND: C5.1.2, LASER_COM-1.S, LASER_COM-2.S, MCU.AVSS, R4.1.1, R4.3.1
- net GND: now also XTL.G2; no longer C5.1.2, LASER_COM-1.S, LASER_COM-2.S, MCU.AVSS, R4.1.1, R4.3.1, XTL.G1
Changed lines of the file:
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@@
-</segment>
-<segment>
-<wire x1="-76.2" y1="187.96" x2="-76.2" y2="205.74" width="0.1524" layer="91"/>
-<pinref part="XTL" gate="G$1" pin="G1"/>
-<wire x1="-76.2" y1="205.74" x2="-76.2" y2="213.36" width="0.1524" layer="91"/>
-<wire x1="-81.28" y1="205.74" x2="-76.2" y2="205.74" width="0.1524" layer="91"/>
-<junction x="-76.2" y="205.74"/>
-<label x="-76.2" y="213.36" size="1.778" layer="95" rot="R90"/>
-<pinref part="MCU" gate="A" pin="AVSS"/>
-<wire x1="-76.2" y1="187.96" x2="-60.96" y2="187.96" width="0.1524" layer="91"/>
-<pinref part="C5.1" gate="G$1" pin="2"/>
 </segment>
 <segment>
@@
 <wire x1="83.82" y1="175.26" x2="88.9" y2="175.26" width="0.1524" layer="91"/>
 <junction x="83.82" y="175.26"/>
-<label x="91.44" y="175.26" size="1.778" layer="95"/>
+<label x="99.06" y="175.26" size="1.778" layer="95"/>
 <pinref part="C5.3" gate="G$1" pin="2"/>
-<wire x1="88.9" y1="175.26" x2="91.44" y2="175.26" width="0.1524" layer="91"/>
+<wire x1="88.9" y1="175.26" x2="96.52" y2="175.26" width="0.1524" layer="91"/>
 <wire x1="88.9" y1="170.18" x2="88.9" y2="175.26" width="0.1524" layer="91"/>
 <junction x="88.9" y="175.26"/>
@@
 </segment>
 <segment>
-<pinref part="U4.1" gate="A" pin="GND"/>
-<wire x1="180.34" y1="93.98" x2="180.34" y2="83.82" width="0.1524" layer="91"/>
-<pinref part="R4.1" gate="G$1" pin="1"/>
-<wire x1="190.5" y1="83.82" x2="180.34" y2="83.82" width="0.1524" layer="91"/>
-<wire x1="180.34" y1="83.82" x2="162.56" y2="83.82" width="0.1524" layer="91"/>
-<junction x="180.34" y="83.82"/>
-<label x="157.48" y="83.82" size="1.778" layer="95" rot="R180"/>
-<pinref part="R4.3" gate="G$1" pin="1"/>
-<wire x1="162.56" y1="83.82" x2="157.48" y2="83.82" width="0.1524" layer="91"/>
-<wire x1="165.1" y1="73.66" x2="162.56" y2="73.66" width="0.1524" layer="91"/>
-<wire x1="162.56" y1="73.66" x2="162.56" y2="83.82" width="0.1524" layer="91"/>
-<junction x="162.56" y="83.82"/>
-</segment>
-<segment>
 <pinref part="JP4" gate="G$1" pin="9"/>
 <wire x1="198.12" y1="157.48" x2="203.2" y2="157.48" width="0.1524" layer="91"/>
@@
 </segment>
 <segment>
-<pinref part="LASER_COM" gate="-2" pin="S"/>
-<wire x1="-246.38" y1="-106.68" x2="-226.06" y2="-106.68" width="0.1524" layer="91"/>
-<label x="-226.06" y="-106.68" size="1.778" layer="95"/>
-</segment>
-<segment>
-<pinref part="LASER_COM" gate="-1" pin="S"/>
-<wire x1="-246.38" y1="-109.22" x2="-226.06" y2="-109.22" width="0.1524" layer="91"/>
-<label x="-226.06" y="-109.22" size="1.778" layer="95"/>
-</segment>
-<segment>
 <pinref part="R1.1" gate="G$1" pin="1"/>
 <wire x1="-205.74" y1="187.96" x2="-200.66" y2="187.96" width="0.1524" layer="91"/>
@@
 <junction x="-175.26" y="-50.8"/>
 <label x="-175.26" y="-55.88" size="1.778" layer="95"/>
+</segment>
+<segment>
+<pinref part="XTL" gate="G$1" pin="G2"/>
+<wire x1="-91.44" y1="205.74" x2="-99.06" y2="205.74" width="0.1524" layer="91"/>
+<wire x1="-99.06" y1="205.74" x2="-99.06" y2="200.66" width="0.1524" layer="91"/>
+<label x="-99.06" y="200.66" size="1.778" layer="95" rot="R270"/>
+</segment>
+<segment>
+<pinref part="U4.1" gate="A" pin="GND"/>
+<wire x1="180.34" y1="93.98" x2="170.18" y2="93.98" width="0.1524" layer="91"/>
+<label x="167.64" y="93.98" size="1.778" layer="95" rot="R180"/>
 </segment>
 </net>
@@
 <wire x1="78.74" y1="182.88" x2="83.82" y2="182.88" width="0.1524" layer="91"/>
 <pinref part="C5.2" gate="G$1" pin="1"/>
-<wire x1="83.82" y1="182.88" x2="91.44" y2="182.88" width="0.1524" layer="91"/>
+<wire x1="83.82" y1="182.88" x2="96.52" y2="182.88" width="0.1524" layer="91"/>
 <junction x="83.82" y="182.88"/>
-<label x="91.44" y="182.88" size="1.778" layer="95"/>
+<label x="99.06" y="182.88" size="1.778" layer="95"/>
 </segment>
 <segment>
@@
 </segment>
 </net>
+<net name="A_GND" class="0">
+<segment>
+<wire x1="-76.2" y1="187.96" x2="-76.2" y2="205.74" width="0.1524" layer="91"/>
+<wire x1="-76.2" y1="205.74" x2="-76.2" y2="213.36" width="0.1524" layer="91"/>
+<junction x="-76.2" y="205.74"/>
+<label x="-76.2" y="213.36" size="1.778" layer="95" rot="R90"/>
+<pinref part="MCU" gate="A" pin="AVSS"/>
+<wire x1="-76.2" y1="187.96" x2="-60.96" y2="187.96" width="0.1524" layer="91"/>
+<pinref part="C5.1" gate="G$1" pin="2"/>
+</segment>
+<segment>
+<pinref part="R4.1" gate="G$1" pin="1"/>
+<wire x1="190.5" y1="83.82" x2="162.56" y2="83.82" width="0.1524" layer="91"/>
+<label x="157.48" y="83.82" size="1.778" layer="95" rot="R180"/>
+<pinref part="R4.3" gate="G$1" pin="1"/>
+<wire x1="162.56" y1="83.82" x2="157.48" y2="83.82" width="0.1524" layer="91"/>
+<wire x1="165.1" y1="73.66" x2="162.56" y2="73.66" width="0.1524" layer="91"/>
+<wire x1="162.56" y1="73.66" x2="162.56" y2="83.82" width="0.1524" layer="91"/>
+<junction x="162.56" y="83.82"/>
+</segment>
+<segment>
+<pinref part="LASER_COM" gate="-2" pin="S"/>
+<wire x1="-246.38" y1="-106.68" x2="-226.06" y2="-106.68" width="0.1524" layer="91"/>
+<label x="-226.06" y="-106.68" size="1.778" layer="95"/>
+</segment>
+<segment>
+<pinref part="LASER_COM" gate="-1" pin="S"/>
+<wire x1="-246.38" y1="-109.22" x2="-226.06" y2="-109.22" width="0.1524" layer="91"/>
+<label x="-226.06" y="-109.22" size="1.778" layer="95"/>
+</segment>
+</net>

Commit message: Analog ground isolation
Moved opamp to Agnd
added Agnd plane
Added decoupling cap to opamp
Parts:
- added C4.1: 10 uF, adafruit:C-USC1206
Connections:
- net A_GND: now also C4.1.1, U4.1.GND
- net GND: no longer U4.1.GND
- net VCC_3V: now also C4.1.2
Other:
- note added: "Laser Connector ---------------------------------------- Provides data link to laser"
- note removed: "Laser Connector ---------------------------------------- DB25 connector sourcing power and data to laser. Must source/sink 10A @5V"
Changed lines of the file:
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@@
 <part name="LED9.1" library="led" deviceset="LED" device="SMT1206"/>
 <part name="R9.4" library="adafruit" deviceset="R-US_" device="M1206" value="100k"/>
+<part name="C4.1" library="adafruit" deviceset="C-US" device="C1206" value="10 uF"/>
 </parts>
 <sheets>
@@
 <text x="-256.54" y="-88.9" size="1.778" layer="97">Laser Connector
 ----------------------------------------
-DB25 connector sourcing power and data to laser.
-Must source/sink 10A @5V</text>
+Provides data link to laser</text>
 <text x="-101.6" y="-81.28" size="1.778" layer="97">LCD interface
 -------------------------------------------------
@@
 <instance part="LED9.1" gate="G$1" x="-50.8" y="-50.8"/>
 <instance part="R9.4" gate="G$1" x="-55.88" y="-58.42"/>
+<instance part="C4.1" gate="G$1" x="167.64" y="91.44" smashed="yes" rot="R180">
+<attribute name="NAME" x="164.084" y="90.805" size="1.778" layer="95" rot="R180"/>
+<attribute name="VALUE" x="166.624" y="88.011" size="1.778" layer="96" rot="R180"/>
+</instance>
 </instances>
 <busses>
@@
 <wire x1="-99.06" y1="205.74" x2="-99.06" y2="200.66" width="0.1524" layer="91"/>
 <label x="-99.06" y="200.66" size="1.778" layer="95" rot="R270"/>
-</segment>
-<segment>
-<pinref part="U4.1" gate="A" pin="GND"/>
-<wire x1="180.34" y1="93.98" x2="170.18" y2="93.98" width="0.1524" layer="91"/>
-<label x="167.64" y="93.98" size="1.778" layer="95" rot="R180"/>
 </segment>
 </net>
@@
 <label x="223.52" y="190.5" size="1.778" layer="95"/>
 </segment>
+<segment>
+<pinref part="C4.1" gate="G$1" pin="2"/>
+<wire x1="167.64" y1="96.52" x2="157.48" y2="96.52" width="0.1524" layer="91"/>
+<label x="154.94" y="96.52" size="1.778" layer="95" rot="R180"/>
+</segment>
 </net>
 <net name="N$11" class="0">
@@
 <segment>
 <pinref part="U4.1" gate="A" pin="1OUT"/>
-<wire x1="180.34" y1="101.6" x2="170.18" y2="101.6" width="0.1524" layer="91"/>
+<wire x1="180.34" y1="101.6" x2="162.56" y2="101.6" width="0.1524" layer="91"/>
 <pinref part="U4.1" gate="A" pin="1IN-"/>
 <wire x1="180.34" y1="99.06" x2="180.34" y2="101.6" width="0.1524" layer="91"/>
 <junction x="180.34" y="101.6"/>
-<label x="170.18" y="101.6" size="1.778" layer="95" rot="R180"/>
+<label x="157.48" y="101.6" size="1.778" layer="95" rot="R180"/>
 </segment>
 </net>
@@
 <segment>
 <pinref part="R4.1" gate="G$1" pin="1"/>
-<wire x1="190.5" y1="83.82" x2="162.56" y2="83.82" width="0.1524" layer="91"/>
+<wire x1="190.5" y1="83.82" x2="180.34" y2="83.82" width="0.1524" layer="91"/>
 <label x="157.48" y="83.82" size="1.778" layer="95" rot="R180"/>
 <pinref part="R4.3" gate="G$1" pin="1"/>
+<wire x1="180.34" y1="83.82" x2="167.64" y2="83.82" width="0.1524" layer="91"/>
+<wire x1="167.64" y1="83.82" x2="162.56" y2="83.82" width="0.1524" layer="91"/>
 <wire x1="162.56" y1="83.82" x2="157.48" y2="83.82" width="0.1524" layer="91"/>
 <wire x1="165.1" y1="73.66" x2="162.56" y2="73.66" width="0.1524" layer="91"/>
 <wire x1="162.56" y1="73.66" x2="162.56" y2="83.82" width="0.1524" layer="91"/>
 <junction x="162.56" y="83.82"/>
-</segment>
-<segment>
+<pinref part="U4.1" gate="A" pin="GND"/>
+<wire x1="180.34" y1="93.98" x2="180.34" y2="83.82" width="0.1524" layer="91"/>
+<junction x="180.34" y="83.82"/>
+<pinref part="C4.1" gate="G$1" pin="1"/>
+<wire x1="167.64" y1="88.9" x2="167.64" y2="83.82" width="0.1524" layer="91"/>
+<junction x="167.64" y="83.82"/>
+</segment>
+<segment>

Commit message: Updated Schematic.
Updated schematic layout. Added frame, updated passive components, set
(some) resistor values.
Parts:
- removed C1.1, C4.1, C6.3, C8.4: 10 uF, adafruit:C-USC1206
- removed C1.2, C1.4, C5.2, C5.3, C5.4, C6.4, C6.5, C8.10, C8.3, C8.9: 0.1 uF, adafruit:C-USC1206
- removed C1.3: 0.01 uF, adafruit:C-USC1206
- removed C6.1, C8.1, C9.1: 4.7 uF, adafruit:C-USC1206
- removed C6.2, C8.2, C9.2, C9.3: 2.2 uF, adafruit:C-USC1206
- removed C7.1: 2.2 nF, adafruit:C-USC1206
- removed C8.5, C8.6, C8.7, C8.8: 1 uF, adafruit:C-USC1206
- removed D1: (no value), adafruit:DIODESOD-123
- removed L6.1, L8.1, L9.1: 3 uH, adafruit:FB
- removed R1.1, R7.1: 47k, adafruit:R-US_M1206
- removed R2.1: 10k, adafruit:R-US_M1206
- removed R2.2: (no value), adafruit:R-US_M1206
- removed R4.1: 1M, adafruit:R-US_R1206
- removed R4.2: 0R, adafruit:R-US_R1206
- removed R4.3: 600k, adafruit:R-US_R1206
- removed R4.4: 400k, adafruit:R-US_R1206
- removed R5.1, R5.2: 43k, adafruit:R-US_M1206
- removed R8.1, R8.2, R8.3, R8.4, R9.4: 100k, adafruit:R-US_M1206
- removed R9.2: 500k, adafruit:R-US_M1206
- removed U4.1: TLV2242_D_8, TI:TLV2242_D_8
- added C1, C11, C12, C13, C16, C18, C2, C23, C27, C3, C6, C7, C8: .1uF, rc-master-smd:C_0603
- added C10, C17, C26, C5: 10uF, rc-master-smd:C_0603
- added C14, C15: 1uF, rc-master-smd:C_0603
- added C19, C21, C24: 2.2uF, rc-master-smd:C_0603
- added C20, C22, C25: 4.7uF, rc-master-smd:C_0603
- added C4: 2.2nF, rc-master-smd:C_0603
- added C9: .01uF, rc-master-smd:C_0603
- added D2: BAR43, diode:BAR43
- added L1, L2, L3: 3uH, rc-master-smd:L_0805
- added R1, R3: 1.2K, rc-master-smd:R_0603
- added R10, R11, R12, R13, R6, R9: 330, rc-master-smd:R_0603
- added R2: 47K, rc-master-smd:R_0603
- added R4: 600K, rc-master-smd:R_0603
- added R5: 400K, rc-master-smd:R_0603
- added R7: 10K, rc-master-smd:R_0603
- added R8: (no value), rc-master-smd:R_0603
- added U1: TLV2242_D_8, op-amp:LMV358D
- C5.1: device adafruit:C-USC1206 -> rc-master-smd:C_0603
- R9.3: value 500k -> 1.2K
Connections:
- net TTL_IN_ISO renamed N$11
- removed net ITL_POWER: C9.2.1, L9.1.2, U9.1.VI+
- removed net N$10: R4.3.2, R4.4.1, U4.1.1IN+
- removed net N$11 (its old number): C6.2.1, L6.1.2, U6.1.VI+
- removed net N$31: LED8.2.C, R8.2.1
- removed net N$35: H9.1.1, R9.2.1
- removed net N$8 (its old number): R4.1.2, R4.2.1, U4.1.2IN+
- removed net SERIAL_GND: C8.3.1, C8.4.1, C8.5.1, C8.8.1, C8.9.2, H8.1.1, U8.1.VO-, U8.2.GND, U8.3.GND2
- removed net SERIAL_VCC: C8.3.2, C8.4.2, C8.9.1, U8.1.VO+, U8.2.VCC, U8.3.VCC2
- removed net VCC_3V: C4.1.2, C5.1.1, C5.2.1, C8.10.1, D1.C, H3.1.3, H7.1.2, MCU.AVCC, MCU.DVCC, R2.1.2, R5.1.1, R5.2.1, R7.1.2, U2.1.VCCI, U4.1.VCC, U8.3.VCC1
- removed net VCC_3V_SUPPLY: C1.4.1, D1.A, U1.1.VOUT
- new net +3V3: C1.1, C11.1, C16.2, C5.1.1, C6.2, D2.A, H3.1.3, H7.1.2, MCU.AVCC, MCU.DVCC, R1.1, R2.2, R3.1, R7.2, U1.1.VOUT, U1P.V+, U2.1.VCCI, U8.3.VCC1
- new net +5V: C10.1, C20.1, C22.1, C23.2, C25.1, C27.2, C3.1, C7.1, C8.2, D2.C, EXT_POWER-1.KL, H6.1.8, H8.2.1, L1.2, L2.2, L3.2, LED1.A, MCU.DVIO, R8.2, U1.1.ENABLE, U1.1.VIN, U2.1.ADDR, U2.1.VCCP, U6.2.VCC2, U6.3.V+, U6.4.V+, U9.2.VCC2, VR1.E
- new net N$18: R4.1, R5.1, U1A.+IN
- new net N$20: LED1.C, R6.2
- new net N$23: LED8.1.C, R9.2
- new net N$32: C24.1, L3.1, U6.1.VI+
- new net SGND: C12.1, C13.1, C17.2, C18.2, H8.1.1, U8.1.VO-, U8.2.GND, U8.3.GND2
- new net VBUS: C17.1, C18.1, U8.1.VO+, U8.2.VCC, U8.3.VCC2
- net A_GND: no longer C4.1.1, C5.1.2, MCU.AVSS, R4.1.1, R4.3.1, U4.1.GND
- net GND: now also C1.2, C10.2, C11.2, C16.1, C19.2, C2.2, C20.2, C21.2, C22.2, C23.1, C24.2, C25.2, C27.1, C3.2, C4.2, C5.1.2, C6.1, C7.2, C8.1, C9.2, MCU.AVSS, R10.1, R11.1, R12.1, R13.2, R4.2, R6.1, R9.1, U1P.GND, U9.2.GND2, XTL.G1; no longer C1.1.2, C1.2.2, C1.3.2, C1.4.2, C5.2.2, C5.3.2, C5.4.2, C6.1.2, C6.2.2, C6.5.1, C7.1.2, C8.1.2, C8.10.2, C8.2.2, C9.1.2, C9.2.2, LED8.1.C, R1.1.1, R8.2.2, R8.3.1, R8.4.1, R9.4.1, U9.2.VCC2
- net LASER_CURRENT: now also R5.2; no longer R4.4.2
- net LASER_CURRENT_3V: now also U1A.-IN, U1A.OUT; no longer U4.1.1IN-, U4.1.1OUT
- net LASER_TEMPERATURE: now also U1B.+IN; no longer R4.2.2
- net LASER_TEMPERATURE_3V: now also U1B.-IN, U1B.OUT; no longer U4.1.2IN-, U4.1.2OUT
- net N$1: now also C14.1, U8.2.C2+; no longer C8.6.1, U8.2.C1+
- net N$13: now also C9.1; no longer C1.3.1
- net N$15: now also R7.1; no longer R2.1.1
- net N$2: now also C14.2, U8.2.C2-; no longer C8.6.2, U8.2.C1-
- net N$24: now also C2.1; no longer C5.3.1
- net N$25: now also LED8.2.C, R10.2; no longer LED1.C, R1.1.2
- net N$26: now also LED8.4.C, R11.2; no longer LED8.3.C, R8.3.2
- net N$27: now also C26.2, H9.1.1; no longer C9.3.1, R9.2.2
- net N$28: now also C26.1; no longer C9.3.2
- net N$29: now also LED8.3.C, R12.2; no longer LED8.4.C, R8.4.2
- net N$3: now also C15.1, U8.2.C1-; no longer C8.7.1, U8.2.C2+
- net N$30: now also R13.1; no longer R9.4.2
- net N$33: now also C19.1, L1.1, U8.1.VI+; no longer LED8.1.A, R8.1.2
- net N$4: now also C15.2, U8.2.C1+; no longer C8.7.2, U8.2.C2-
- net N$5: now also C13.2; no longer C8.8.2
- net N$6: now also C12.2; no longer C8.5.2
- net N$9: now also C21.1, L2.1, U9.1.VI+; no longer C8.2.1, L8.1.2, U8.1.VI+
- net RST: now also C4.1, R2.1; no longer C7.1.1, R7.1.1
- net SCL: now also R3.2; no longer R5.1.2
- net SDA: now also R1.2; no longer R5.2.2
- net TTL_GND_ISO: now also C5.1; no longer C6.3.2, C6.4.2
- net TTL_ISO_VCC: now also C5.2; no longer C6.3.1, C6.4.1
- net TX1: now also LED8.1.A; no longer R8.1.1
- net VCC_5V: no longer C1.1.1, C1.2.1, C5.4.1, C6.1.1, C6.5.2, C8.1.1, C9.1.1, EXT_POWER-1.KL, H6.1.8, H8.2.1, L6.1.1, L8.1.1, L9.1.1, LED1.A, MCU.DVIO, R2.2.2, U1.1.ENABLE, U1.1.VIN, U2.1.ADDR, U2.1.VCCP, U6.2.VCC2, U6.3.V+, U6.4.V+, U9.2.GND2, VR1.E
- net VCC_LED: now also R8.1; no longer R2.2.1
Other:
- note removed: "I2C Pull up ----------------------------"
- moved on the sheet: EXT_POWER-1, EXT_POWER-2, H2.1, H3.1, H6.1, H6.2-1, H6.2-2, H7.1, H8.1, H8.2, H9.1, JP4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
