File: pcb.sch (EAGLE design)
At the start: 81 parts, among them U1 TLV2242_D_8, U1.1 REG101-3_DBV_5, U2.1 TCA6416A_PW_24, U6.1 DCH010505S_EDJ_4, U6.2 ISO7221A_D_8, U6.3 TS5A3357_DCU_8, U6.4 TS5A3357_DCU_8, U8.1 DCH010505S_EDJ_4, U8.2 MAX232E_D_16, U8.3 ISO7221A_D_8, U9.1 DCH010505S_EDJ_4, U9.2 ISO7420Fx

Commit message: Reliability Changes
Changed oscillator circuit, changed voltage regulator to larger package
(current capability), added TVS diodes and current limiting resistors to
I/O. Updated schematic layout.
Parts:
- removed C9: .01uF, rc-master-smd:C_0603
- removed U1.1: REG101-3_DBV_5, TI:REG101-3_DBV_5
- removed XTL: (no value), adafruit:XTAL-4-3225
- added C28: 10uF, rc-master-smd:C_0603
- added C29, C30: 22pF, rc-master-smd:C_0603
- added C31: 4.7uF, rc-master-smd:C_0603
- added C32: .1uF, rc-master-smd:C_0603
- added D1: BAS70, diode:BAS70
- added D3, D4, D5, D6: SRV05-4, diode:SRV05-4
- added R14, R15, R16, R17, R18, R19, R20, R21: 330, rc-master-smd:R_0603
- added U2: LT1117-S, v-reg:LT1117-S
- added Y1: 16MHZ, crystal:CRYTALHC49S
- C2: value .1uF -> .47uF
- D2: value BAR43 -> SRV05-4; device diode:BAR43 -> diode:SRV05-4
- R9.1: value 100k -> 47K
Connections:
- removed net A_GND: LASER_COM-1.S, LASER_COM-2.S
- removed net VCC_5V: H2.1.2
- new net N$10: LASER_COM-3.S, R17.2
- new net N$31: LASER_COM-5.S, R15.2
- new net N$34: LASER_COM-6.S, R14.2
- new net N$35: R21.1
- new net N$36: R18.1
- new net N$37: R19.1
- new net N$38: R20.1
- net +3V3: now also C28.1, C31.1, C32.2, D1.A, D2.5, D3.5, D5.5, U2.OUT, U2.TAB; no longer D2.A, U1.1.VOUT
- net +5V: now also D1.C, D4.5, D6.5, H2.1.2, U2.IN; no longer D2.C, U1.1.ENABLE, U1.1.VIN
- net 3VIO-0H: now also D3.1
- net 3VIO-1H: now also D3.3
- net 3VIO-2H: now also D3.4
- net 3VIO-3H: now also D2.6
- net 3VIO-4H: now also D2.1
- net 3VIO-5H: now also D2.3
- net 3VIO-6H: now also D2.4
- net 5VIO-0: now also D4.4, R20.2
- net 5VIO-1: now also D4.3, R19.2
- net 5VIO-2: now also D4.1, R18.2
- net 5VIO-3: now also D4.6, R21.2
- net GND: now also C28.2, C29.2, C30.2, C31.2, C32.1, D2.2, D3.2, D4.2, D5.2, D6.2, LASER_COM-1.S, LASER_COM-2.S, U2.GND; no longer C9.2, U1.1.GND, XTL.G1, XTL.G2
- net LASER_CURRENT: now also D6.3, R16.1; no longer LASER_COM-4.S
- net LASER_ILK: now also D6.6, R14.1; no longer LASER_COM-6.S
- net LASER_TEMPERATURE: now also D6.4, R17.1; no longer LASER_COM-3.S
- net LASER_TTL: now also D6.1, R15.1; no longer LASER_COM-5.S
- net N$13: now also LASER_COM-4.S, R16.2; no longer C9.1, U1.1.NR/ADJUST
- net N$21: now also C29.1, Y1.2; no longer XTL.X1
- net N$22: now also C30.1, Y1.1; no longer XTL.X2
- net SCL: now also D5.4
- net SDA: now also D5.3
Other:
- moved on the sheet: C1, C10, C11, C12, C13, C14, C15, C16, C17, C18, C19, C2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

Commit message: Connector Update
Added DB25 laser connector and replaced power connector with mini-fit
Jr. Added logic buffer to laser outputs. Minor additional updates.
Parts:
- removed C3.1: 100 nF, TI:468M-801-XXX
- removed D6: SRV05-4, diode:SRV05-4
- removed EXT_POWER: (no value), con-wago-500:W237-102
- removed H7.1: (no value), jumper:JP2E
- removed LASER_COM: C-GRID-06-70553, con-molex:C-GRID-06-70553
- removed R14, R15, R16, R17: 330, rc-master-smd:R_0603
- added C33, C34, C35, C36, C37, C38, C39, C40, C9: .1uF, rc-master-smd:C_0603
- added CN1: NC182M25, custom:NC182M25
- added H9.2: (no value), jumper:JP2E
- added P1: 39-30-02, con-molex-mini-fit:39-30-02
- added R22: 330, rc-master-smd:R_0603
- added U3, U4: SN74LVC1G17DBV, 74LV:SN74LVC1G17DBV
- R8: value (none) -> 0
- U9.2: value ISO7420Fx -> ISO7220D
Connections:
- net VCC_LED renamed N$41
- removed net N$17: H7.1.3, JP4.2
- removed net N$31: LASER_COM-5.S, R15.2
- removed net N$34: LASER_COM-6.S, R14.2
- removed net N$35: R21.1
- removed net N$36: R18.1
- removed net N$37: R19.1
- removed net N$38: R20.1
- new net 5VIO-4: D4.4, R20.1
- new net N$12: CN1.1, U3.Y
- new net N$39: R22.2, VR1.E
- net +3V3: now also H9.2.2; no longer H7.1.2
- net +5V: now also C39.1, C40.1, CN1.10, CN1.11, CN1.12, CN1.13, CN1.5, CN1.6, CN1.7, CN1.8, CN1.9, P1.2, R22.1, U3.VCC, U4.VCC; no longer D6.5, EXT_POWER-1.KL, VR1.E
- net 3VIO-0H: now also C9.1; no longer C3.1.1
- net 3VIO-1H: now also C33.1; no longer C3.1.2
- net 3VIO-2H: now also C34.1; no longer C3.1.3
- net 3VIO-3H: now also C35.1; no longer C3.1.4
- net 3VIO-4H: now also C36.1; no longer C3.1.5
- net 3VIO-5H: now also C37.1; no longer C3.1.6
- net 3VIO-6H: now also C38.1; no longer C3.1.7
- net 5VIO-0: no longer D4.4
- net 5VIO-1: now also D4.6, R21.1; no longer D4.3
- net 5VIO-2: now also R18.1
- net 5VIO-3: now also D4.3, R19.1; no longer D4.6
- net GND: now also C33.2, C34.2, C35.2, C36.2, C37.2, C38.2, C39.2, C40.2, C9.2, CN1.17, CN1.18, CN1.19, CN1.20, CN1.21, CN1.22, CN1.23, CN1.24, CN1.25, CN1.G1, CN1.G2, P1.1, U3.GND, U4.GND; no longer C3.1.BUS, C3.1.BUS2, D6.2, EXT_POWER-2.KL, LASER_COM-1.S, LASER_COM-2.S
- net LASER_CURRENT: now also CN1.2; no longer D6.3, R16.1
- net LASER_ILK: now also U3.A; no longer D6.6, R14.1
- net LASER_TEMPERATURE: now also CN1.3; no longer D6.4, R17.1
- net LASER_TTL: now also U4.A; no longer D6.1, R15.1
- net N$10: now also CN1.14, U4.Y; no longer LASER_COM-3.S, R17.2
- net N$13: now also H9.2.1, JP4.4; no longer LASER_COM-4.S, R16.2
- net N$16: now also H9.2.3, JP4.2; no longer H7.1.1, JP4.4
Other:
- note added: "A"
- note added: "Laser Connector ---------------------------------------- Provides data link and power to the laser"
- note added: "Laser Controller"
- note removed: "100 nF"
- note removed: "Laser Connector ---------------------------------------- Provides data link to laser"
- moved on the sheet: C10, C4, C7, D2, D3, D4, D5, H3.1, H6.1, R1, R18, R19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

Commit message: Routing complete
All placement complete and signals routed. Awaiting copper planes,
renaming components, name placement and silkscreen.
Parts:
- removed R9.1: 47K, adafruit:R-US_M1206
- removed R9.3: 1.2K, adafruit:R-US_M1206
- added R14: 47K, rc-master-smd:R_0603
- added R15: 1.2K, rc-master-smd:R_0603
Connections:
- removed net 5VIO-4: D4.4, R20.1
- new net N$17: H6.1.1, R21.2
- new net N$31: H6.1.3, R18.2
- new net N$34: H6.1.5, R19.2
- new net N$35: H6.1.7, R20.2
- net 3VIO-0H: now also D3.4; no longer D3.1
- net 3VIO-2H: now also D3.1; no longer D3.4
- net 3VIO-3H: now also D2.4; no longer D2.6
- net 3VIO-4H: now also D2.3; no longer D2.1
- net 3VIO-5H: now also D2.1; no longer D2.3
- net 3VIO-6H: now also D2.6; no longer D2.4
- net 5VIO-0: now also D4.1, R21.1; no longer H6.1.7, R20.2
- net 5VIO-1: now also R18.1; no longer H6.1.5, R19.2, R21.1
- net 5VIO-2: now also D4.4, R19.1; no longer D4.1, H6.1.3, R18.1, R18.2
- net 5VIO-3: now also R20.1; no longer H6.1.1, R19.1, R21.2
- net LASER_CURRENT_3V: now also MCU.P1.3/PM_UCB0CLK/PM_UCA0STE/A3*/CB3; no longer MCU.P1.0/PM_UCA0CLK/PM_UCB0STE/A0*/CB0
- net LASER_ILK: now also R14.2; no longer R9.1.2
- net LASER_ILK_HIGH: now also R14.1; no longer R9.1.1
- net LASER_TEMPERATURE_3V: now also MCU.P1.0/PM_UCA0CLK/PM_UCB0STE/A0*/CB0; no longer MCU.P1.3/PM_UCB0CLK/PM_UCA0STE/A3*/CB3
- net N$14: now also R15.2; no longer R9.3.1
- net N$19: now also R15.1; no longer R9.3.2

Commit message: Copper Pours & Component Silk Complete
Poured Copper planes and adjusted component designators for proper
silkscreen printing. Renumbered components.
Parts:
- removed R21, R22: 330, rc-master-smd:R_0603
- added R16, R17: 330, rc-master-smd:R_0603
- C1: value .1uF -> 22pF
- C10, C5: value 10uF -> .1uF
- C14: value 1uF -> 10uF
- C15: value 1uF -> .1uF
- C17, C26: value 10uF -> 4.7uF
- C19: value 2.2uF -> .47uF
- C2: value .47uF -> 22pF
- C20, C22, C31: value 4.7uF -> .1uF
- C21: value 2.2uF -> .1uF
- C23: value .1uF -> 2.2nF
- C24: value 2.2uF -> 4.7uF
- C27: value .1uF -> 2.2uF
- C28: value 10uF -> 2.2uF
- C29: value 22pF -> 2.2uF
- C30: value 22pF -> .1uF
- C34, C37, C40: value .1uF -> 10uF
- C35, C36: value .1uF -> 1uF
- C4: value 2.2nF -> 10uF
- D1: value BAS70 -> SRV05-4; device diode:BAS70 -> diode:SRV05-4
- D2: value SRV05-4 -> BAS70; device diode:SRV05-4 -> diode:BAS70
- H8.1: device jumper:JP2E -> jumper:JP4E
- H8.2: device jumper:JP4E -> jumper:JP2E
- R1, R15: value 1.2K -> 330
- R2: value 47K -> 400K
- R20: value 330 -> 1.2K
- R3: value 1.2K -> 600K
- R4: value 600K -> 1.2K
- R5: value 400K -> 1.2K
- R6: value 330 -> 10K
- R7: value 10K -> 330
- R9: value 330 -> 47K
- U1: value TLV2242_D_8 -> LT1117-S; device op-amp:LMV358D -> v-reg:LT1117-S
- U2: value LT1117-S -> TLV2242_D_8; device v-reg:LT1117-S -> op-amp:LMV358D
- U6.1: value DCH010505S_EDJ_4 -> TS5A3357_DCU_8; device TI:DCH010505S_EDJ_4 -> TI:TS5A3357_DCU_8
- U6.2: value ISO7221A_D_8 -> TS5A3357_DCU_8; device TI:ISO7221A_D_8 -> TI:TS5A3357_DCU_8
- U6.3: value TS5A3357_DCU_8 -> DCH010505S_EDJ_4; device TI:TS5A3357_DCU_8 -> TI:DCH010505S_EDJ_4
- U6.4: value TS5A3357_DCU_8 -> ISO7221A_D_8; device TI:TS5A3357_DCU_8 -> TI:ISO7221A_D_8
- U8.2: value MAX232E_D_16 -> ISO7221A_D_8; device TI:MAX232E_D_16 -> TI:ISO7221A_D_8
- U8.3: value ISO7221A_D_8 -> MAX232E_D_16; device TI:ISO7221A_D_8 -> TI:MAX232E_D_16
- renumbered JP4 to JP1
Connections:
- net +3V3: now also C13.1, C14.1, C15.2, C17.1, C18.1, C3.2, C30.2, D1.5, D2.A, D4.5, H9.1.2, R4.1, R5.1, R6.2, R9.2, U1.OUT, U1.TAB, U2P.V+, U8.2.VCC1; no longer C1.1, C11.1, C16.2, C28.1, C31.1, C32.2, C6.2, D1.A, D2.5, D5.5, H9.2.2, R1.1, R2.2, R3.1, R7.2, U1P.V+, U2.OUT, U2.TAB, U8.3.VCC1
- net +5V: now also C16.1, C21.2, C24.1, C26.1, C31.2, C32.2, C4.1, D2.C, D5.5, H8.1.1, R7.1, U1.IN, U6.1.V+, U6.2.V+, U6.4.VCC2; no longer C10.1, C23.2, C27.2, C3.1, C39.1, C40.1, C8.2, D1.C, D4.5, H8.2.1, R22.1, U2.IN, U6.2.VCC2, U6.3.V+, U6.4.V+
- net 3VIO-0H: now also C5.1; no longer C9.1
- net 3VIO-1H: now also C6.1; no longer C33.1
- net 3VIO-2H: now also C8.1; no longer C34.1
- net 3VIO-3H: now also C9.1, D1.4; no longer C35.1, D2.4
- net 3VIO-4H: now also C10.1, D1.3; no longer C36.1, D2.3
- net 3VIO-5H: now also C11.1, D1.1; no longer C37.1, D2.1
- net 3VIO-6H: now also C12.1, D1.6; no longer C38.1, D2.6
- net 5VIO-0: now also D5.1, R10.1; no longer D4.1, R21.1
- net 5VIO-1: now also D5.6, R11.1; no longer D4.6, R18.1
- net 5VIO-2: now also D5.4, R12.1; no longer D4.4, R19.1
- net 5VIO-3: now also D5.3, R13.1; no longer D4.3, R20.1
- net EXT_SRC-A: now also U6.2.IN1; no longer U6.4.IN1
- net EXT_SRC-B: now also U6.2.IN2; no longer U6.4.IN2
- net EXT_TTL: now also U6.1.NO1, U6.2.NO1; no longer U6.3.NO1, U6.4.NO1
- net GND: now also C12.2, C13.2, C14.2, C15.1, C16.2, C17.2, C18.2, C21.1, C23.2, C26.2, C27.2, C3.1, C30.1, C31.1, C5.2, C6.2, C8.2, D1.2, H8.1.2, R1.1, R15.1, R16.1, R17.2, R18.1, R19.1, R3.2, U1.GND, U2P.GND, U6.1.GND, U6.2.GND, U6.3.VI-, U6.4.GND2, U8.2.GND1; no longer C16.1, C21.2, C23.1, C27.1, C3.2, C30.2, C31.2, C33.2, C34.2, C35.2, C36.2, C37.2, C38.2, C39.2, C40.2, C6.1, C8.1, D2.2, H8.2.2, R10.1, R11.1, R12.1, R13.2, R4.2, R6.1, R9.1, U1P.GND, U2.GND, U6.1.VI-, U6.2.GND2, U6.3.GND, U6.4.GND, U8.3.GND1
- net LASER_CURRENT: now also R2.2; no longer R5.2
- net LASER_CURRENT_3V: now also U2A.-IN, U2A.OUT; no longer U1A.-IN, U1A.OUT
- net LASER_SRC-A: now also U6.1.IN1; no longer U6.3.IN1
- net LASER_SRC-B: now also U6.1.IN2; no longer U6.3.IN2
- net LASER_TEMPERATURE: now also U2B.+IN; no longer U1B.+IN
- net LASER_TEMPERATURE_3V: now also U2B.-IN, U2B.OUT; no longer U1B.-IN, U1B.OUT
- net LASER_TTL: now also U6.1.COM; no longer U6.3.COM
- net MCU_TTL1: now also U6.1.NO0, U6.2.NO2; no longer U6.3.NO0, U6.4.NO2
- net MCU_TTL2: now also U6.2.NO0; no longer U6.4.NO0
- net N$1: now also C36.1, U8.3.C2+; no longer C14.1, U8.2.C2+
- net N$11: now also U6.4.INB; no longer U6.2.INB
- net N$13: now also H9.1.1; no longer H9.2.1
- net N$14: now also H9.2.2, R20.2; no longer H9.1.2, R15.2
- net N$15: now also R6.1; no longer R7.1
- net N$16: now also H9.1.3; no longer H9.2.3
- net N$17: now also R10.2; no longer R21.2
- net N$18: now also R2.1, R3.1, U2A.+IN; no longer R4.1, R5.1, U1A.+IN
- net N$19: now also R20.1; no longer R15.1
- net N$2: now also C36.2, U8.3.C2-; no longer C14.2, U8.2.C2-
- net N$20: now also R1.2; no longer R6.2
- net N$21: now also C1.1; no longer C29.1
- net N$22: now also C2.1; no longer C30.1
- net N$23: now also LED8.2.C, R16.2; no longer LED8.1.C, R9.2
- net N$24: now also C19.1; no longer C2.1
- net N$25: now also LED8.4.C, R19.2; no longer LED8.2.C, R10.2
- net N$26: now also LED8.1.C, R15.2; no longer LED8.4.C, R11.2
- net N$27: now also C34.2, H9.2.1; no longer C26.2, H9.1.1
- net N$28: now also C34.1, H9.2.3; no longer C26.1, H9.1.3
- net N$29: now also R18.2; no longer R12.2
- net N$3: now also C35.1, U8.3.C1-; no longer C15.1, U8.2.C1-
- net N$30: now also R17.1; no longer R13.1
- net N$31: now also R11.2; no longer R18.2
- net N$32: now also C28.1, L2.1, U6.3.VI+; no longer C24.1, L3.1, U6.1.VI+
- net N$33: now also C29.1, L3.1; no longer C19.1, L1.1
- net N$34: now also R12.2; no longer R19.2
- net N$35: now also R13.2; no longer R20.2
- net N$39: now also R7.2; no longer R22.2
- net N$4: now also C35.2, U8.3.C1+; no longer C15.2, U8.2.C1+
- net N$5: now also C39.2, U8.3.VS-; no longer C13.2, U8.2.VS-
- net N$6: now also C38.2, U8.3.VS+; no longer C12.2, U8.2.VS+
- net N$9: now also C27.1, L1.1; no longer C21.1, L2.1
- net RS232_RX: now also H8.2.3, U8.3.RIN1; no longer H8.1.3, U8.2.RIN1
- net RS232_TX: now also H8.2.2, U8.3.DOUT1; no longer H8.1.2, U8.2.DOUT1
- net RST: now also C23.1, R9.1; no longer C4.1, R2.1
- net RX1: now also LED8.4.A, U8.2.OUTA; no longer LED8.2.A, U8.3.OUTA
- net RX2: now also H8.1.4, LED8.1.A; no longer H8.2.4, LED8.4.A
- net SCL: now also D4.4, R5.2; no longer D5.4, R3.2
- net SDA: now also D4.3, R4.2; no longer D5.3, R1.2
- net SERIAL_RX: now also U8.2.INA, U8.3.ROUT1; no longer U8.2.ROUT1, U8.3.INA
- net SERIAL_TX: now also U8.2.OUTB, U8.3.DIN1; no longer U8.2.DIN1, U8.3.OUTB
- net SGND: now also C33.2, C38.1, C39.1, C40.2, H8.2.1, U8.2.GND2, U8.3.GND; no longer C12.1, C13.1, C17.2, C18.2, H8.1.1, U8.2.GND, U8.3.GND2
- net TTL_GND_ISO: now also C37.1, U6.3.VO-, U6.4.GND1; no longer C5.1, U6.1.VO-, U6.2.GND1
- net TTL_IN: now also U6.1.NO2, U6.4.OUTB; no longer U6.2.OUTB, U6.3.NO2
- net TTL_ISO_VCC: now also C37.2, U6.3.VO+, U6.4.VCC1; no longer C5.2, U6.1.VO+, U6.2.VCC1
- net TTL_OUT: now also U6.2.COM, U6.4.INA; no longer U6.2.INA, U6.4.COM
- net TTL_OUT_ISO: now also U6.4.OUTA; no longer U6.2.OUTA
- net TX1: now also LED8.2.A, U8.2.INB; no longer LED8.1.A, U8.3.INB
- net TX2: now also H8.1.3; no longer H8.2.3
- net VBUS: now also C33.1, C40.1, U8.2.VCC2, U8.3.VCC; no longer C17.1, C18.1, U8.2.VCC, U8.3.VCC2
Other:
- moved on the sheet: C1, C10, C11, C12, C13, C14, C15, C16, C17, C18, C19, C2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
